Commit message: Improvements made for faster running Gazebo simulations (smaller triangle count on model and simple collision model for robot). ROS2 Control added and hardware interface and beginnings of the "sim to real" transition taking place.

File: slambot_description/urdf/modules/chassis_and_wheels.xacro (robot description, xacro)
@@ -27,7 +27,7 @@
     </visual>
     <collision>
-      <origin xyz="0 0 0" rpy="0 -0 0"/>
+      <origin xyz="0 0 0.051" rpy="0 -0 0"/>
       <geometry>
-        <mesh filename="package://slambot_description/assets/base_link.stl"/>
+        <box size="0.216 0.156 0.108"/>
       </geometry>
     </collision>
@@ -51,7 +51,7 @@
     </visual>
     <collision>
-      <origin xyz="0 0 0.032" rpy="-1.5708 -0 0"/>
+      <origin xyz="0 0 0.0185" rpy="0 -0 0"/>
       <geometry>
-        <mesh filename="package://slambot_description/assets/wheel_link.stl"/>
+        <cylinder radius="0.034" length="0.027" />
       </geometry>
     </collision>
@@ -83,7 +83,7 @@
     </visual>
     <collision>
-      <origin xyz="0 0 -0.032" rpy="1.5708 -0 0"/>
+      <origin xyz="0 0 -0.0185" rpy="0 -0 0"/>
       <geometry>
-        <mesh filename="package://slambot_description/assets/wheel_link.stl"/>
+        <cylinder radius="0.034" length="0.027" />
       </geometry>
     </collision>
@@ -115,7 +115,7 @@
     </visual>
     <collision>
-      <origin xyz="0 0 -0.032" rpy="1.5708 -0 0"/>
+      <origin xyz="0 0 -0.0185" rpy="0 -0 0"/>
       <geometry>
-        <mesh filename="package://slambot_description/assets/wheel_link.stl"/>
+        <cylinder radius="0.034" length="0.027" />
       </geometry>
     </collision>
@@ -147,7 +147,7 @@
     </visual>
     <collision>
-      <origin xyz="0 0 0.032" rpy="-1.5708 -0 0"/>
+      <origin xyz="0 0 0.0185" rpy="0 -0 0"/>
       <geometry>
-        <mesh filename="package://slambot_description/assets/wheel_link.stl"/>
+        <cylinder radius="0.034" length="0.027" />
       </geometry>
     </collision>

File: slambot_description/urdf/modules/imu_sim.xacro (robot description, xacro)
@@ -7,6 +7,5 @@
     <parent link="base_link"/>
     <child link="imu_link"/>
-    <!-- Place the IMU physically on the base_link, you can adjust the xyz values -->
-    <origin xyz="0 0 0.06" rpy="0 0 0"/>
+    <origin xyz="0 0 0.047" rpy="0 0 0"/>
   </joint>
 </robot>

File: slambot_description/urdf/slambot.urdf.xacro (robot description, xacro)
@@ -3,10 +3,27 @@
 <!-- Onshape document_id: c4aa493c9127ef72e4e641df -->
 <robot name="{robot_name}" xmlns:xacro="http://www.ros.org/wiki/xacro">
+    <xacro:arg name="using_sim" default="true" />
     <xacro:include filename="xacro_properties/xacro_properties.xacro" />
     <xacro:include filename="modules/chassis_and_wheels.xacro" />
     <xacro:include filename="modules/camera.xacro" />
     <xacro:include filename="modules/lidar.xacro" />
-    <xacro:include filename="modules/imu.xacro" />
-    <xacro:include filename="gazebo/gazebo_plugins.xacro" />
-    <xacro:include filename="gazebo/gazebo_properties.xacro" />
+    <xacro:if value="$(arg using_sim)">
+        <xacro:include filename="gazebo/gazebo_plugins.xacro" />
+        <xacro:include filename="modules/imu_sim.xacro" />
+    </xacro:if>
+    <xacro:unless value="$(arg using_sim)">
+        <xacro:include filename="modules/ros2_control.xacro" />
+        <xacro:include filename="modules/imu_real.xacro" />
+    </xacro:unless>
+    <!-- ... inside the launch file ...
+    xacro_file = os.path.join(get_package_share_directory('slambot_description'), 'urdf', 'slambot.urdf.xacro')
+    robot_description_config = Command(['xacro ', xacro_file, ' using_sim:=false'])
+    params = {'robot_description': robot_description_config}
+    node_robot_state_publisher = Node(
+        package='robot_state_publisher',
+        executable='robot_state_publisher',
+        output='screen',
+        parameters=[params]
+    )
+    ... -->
 </robot>
