Commit message: Amendments to launch files and gazebo and RVIZ2 setup

File: slambot_description/urdf/gazebo/gazebo_plugins.xacro (robot description, xacro)
@@ -5,16 +5,28 @@
     <gazebo>
         <plugin filename="gz-sim-diff-drive-system" name="gz::sim::systems::DiffDrive">
-            <left_joint>left_wheel_joint</left_joint>
-            <right_joint>right_wheel_joint</right_joint>
+            <!--wheels-->
+            <left_joint>${robot_name}/left_wheel_joint</left_joint>
+            <right_joint>${robot_name}/right_wheel_joint</right_joint>
+            <!--kinematics-->
             <wheel_separation>0.133</wheel_separation>
             <wheel_radius>0.035</wheel_radius>
+            <!--limits-->
+            <max_linear_acceleration>10</max_linear_acceleration>
+            <!--topics, frames and odometry-->
+            <topic>cmd_vel</topic>
+            <tf_topic>tf</tf_topic>
+            <odom_topic>odom</odom_topic>
             <frame_id>${robot_name}/odom</frame_id> <!--Best to use prefixes and to set the prefix on the RVIZ config too, see xacro_properties.xacro for where to change these -->
             <child_frame_id>${robot_name}/base_footprint</child_frame_id>  <!--Best to use prefixes and to set the prefix on the RVIZ config too, see xacro_properties.xacro for where to change these -->
+            <odom_publisher_frequency>30</odom_publisher_frequency>
         </plugin>
     </gazebo>
     <gazebo>
         <plugin filename="gz-sim-joint-state-publisher-system" name="gz::sim::systems::JointStatePublisher">
-            <joint_name>left_wheel_joint</joint_name>
-            <joint_name>right_wheel_joint</joint_name>
+            <topic>joint_states</topic>
+            <joint_name>${robot_name}/left_wheel_joint</joint_name>
+            <joint_name>${robot_name}/right_wheel_joint</joint_name>
+            <joint_name>${robot_name}/caster_frame_joint</joint_name> <!--Needed, even though not 'driven' joints-->
+            <joint_name>${robot_name}/caster_wheel_joint</joint_name> <!--Needed, even though not 'driven' joints-->
         </plugin>
     </gazebo>
@@ -27,11 +39,12 @@
     </gazebo>
 <!-- =========== Lidar Sensor ============ -->
-    <gazebo reference="lidar_link">
-        <sensor name='gpu_lidar' type='gpu_lidar'>"
-            <pose relative_to='lidar_link'>0 0 0 0 0 0</pose>
+    <gazebo reference="${robot_name}/lidar_link">
+        <sensor name='${robot_name}_lidar' type='gpu_lidar'>
+            <pose relative_to='${robot_name}/lidar_link'>0 0 0 0 0 0</pose>
             <topic>scan</topic>
             <update_rate>2</update_rate>
             <always_on>1</always_on>
             <visualize>1</visualize>
+            <gz_frame_id>${robot_name}/lidar_link</gz_frame_id> <!-- This will give a warning on terminal, but that's a gazebo harmonic issue, so ignore it-->
             <lidar>
                 <scan>
@@ -42,10 +55,4 @@
                         <max_angle>1.396263</max_angle>
                     </horizontal>
-                    <!--<vertical> Not needed if not scanning vertically
-                        <samples>1</samples>
-                        <resolution>0.01</resolution>
-                        <min_angle>0</min_angle>
-                        <max_angle>0</max_angle>
-                    </vertical>-->
                 </scan>
                 <range>
@@ -57,5 +64,5 @@
                     <type>gaussian</type>
                     <mean>0.0</mean>
-                    <stddev>0.001</stddev>
+                    <stddev>0.01</stddev>
                 </noise>
             </lidar>
@@ -64,5 +71,5 @@
 <!--=========================================-->
 <!-- =========== Camera Sensor ============ -->
-    <gazebo reference="camera_mount_link">
+    <gazebo reference="${robot_name}/camera_mount_link">
         <sensor name="camera" type="camera">
             <camera>
@@ -82,5 +89,5 @@
                     <stddev>0.007</stddev>
                 </noise>
-                <optical_frame_id>camera_optical_link</optical_frame_id>
+                <optical_frame_id>${robot_name}/camera_optical_link</optical_frame_id>
                 <camera_info_topic>camera/camera_info</camera_info_topic>
             </camera>

File: slambot_description/urdf/gazebo/gazebo_properties.xacro (robot description, xacro)
@@ -2,13 +2,13 @@
 <robot xmlns:xacro="http://www.ros.org/wiki/xacro">
   <!-- Gazebo properties for the base link -->
-  <gazebo reference="chassis_link">
+  <gazebo reference="${robot_name}/chassis_link">
     <mu1 value="0.5"/> <!-- Friction coefficient in the first direction -->
     <mu2 value="0.5"/> <!-- Friction coefficient in the second direction -->
   </gazebo>
-  <gazebo reference="lidar_link">
+  <gazebo reference="${robot_name}/lidar_link">
     <mu1 value="0.5"/> <!-- Friction coefficient in the first direction -->
     <mu2 value="0.5"/> <!-- Friction coefficient in the second direction -->
   </gazebo>
-  <gazebo reference="camera_mount_link">
+  <gazebo reference="${robot_name}/camera_mount_link">
     <mu1 value="0.5"/> <!-- Friction coefficient in the first direction -->
     <mu2 value="0.5"/> <!-- Friction coefficient in the second direction -->
@@ -16,5 +16,5 @@
   <!-- Gazebo properties for wheel/axle links -->
   <!-- Right Wheel -->
-  <gazebo reference="right_wheel_link">
+  <gazebo reference="${robot_name}/right_wheel_link">
     <mu1 value="1.0"/> <!-- High Friction coefficient for wheels -->
     <mu2 value="1.0"/> <!-- High Friction coefficient for wheels -->
@@ -23,5 +23,5 @@
   </gazebo>
   <!-- Left Wheel -->
-  <gazebo reference="left_wheel_link">
+  <gazebo reference="${robot_name}/left_wheel_link">
     <mu1 value="1.0"/> <!-- High Friction coefficient for wheels -->
     <mu2 value="1.0"/> <!-- High Friction coefficient for wheels -->
@@ -30,5 +30,5 @@
   </gazebo>
   <!-- Caster Wheel -->
-  <gazebo reference="caster_wheel_link">
+  <gazebo reference="${robot_name}/caster_wheel_link">
     <mu1 value="0.8"/> <!-- High Friction coefficient for wheels -->
     <mu2 value="0.8"/> <!-- High Friction coefficient for wheels -->
@@ -37,5 +37,5 @@
   </gazebo>
   <!-- Caster Frame -->
-  <gazebo reference="caster_frame_link">
+  <gazebo reference="${robot_name}/caster_frame_link">
     <mu1 value="0.1"/> <!-- Low Friction coefficient for frame -->
     <mu2 value="0.1"/> <!-- Low Friction coefficient for frame -->

File: slambot_description/urdf/modules/camera.xacro (robot description, xacro)
@@ -4,5 +4,5 @@
 <robot xmlns:xacro="http://www.ros.org/wiki/xacro">
   <!-- Link camera -->
-  <link name="camera_mount_link">
+  <link name="${robot_name}/camera_mount_link">
     <inertial>
       <origin xyz="0 -5.78241e-19 -0.005" rpy="0 0 0"/>
@@ -28,9 +28,9 @@
   </link>
   <!-- Joint from chassis to camera -->
-  <joint name="camera_mount_joint" type="fixed">
+  <joint name="${robot_name}/camera_mount_joint" type="fixed">
     <!--<origin xyz="0.0875 0 0.0335" rpy="-3.14159 1.5708 0"/>-->
     <origin xyz="0.0875 0 0.0335" rpy="0 0 0"/>
-    <parent link="chassis_link"/>
-    <child link="camera_mount_link"/>
+    <parent link="${robot_name}/chassis_link"/>
+    <child link="${robot_name}/camera_mount_link"/>
     <axis xyz="0 0 1"/>
     <limit effort="100" velocity="100"/>
@@ -40,13 +40,13 @@
   http://www.ros.org/reps/rep-0103.html#suffix-frames
   so that ros and opencv can operate on the camera frame correctly -->
-  <link name="camera_optical_link">
+  <link name="${robot_name}/camera_optical_link">
   </link>
-  <joint name="camera_optical_joint" type="fixed">
+  <joint name="${robot_name}/camera_optical_joint" type="fixed">
       <!-- these values have to be these values otherwise the gazebo camera
           image won't be aligned properly with the frame it is supposedly
           originating from -->
       <origin xyz="0 0 0" rpy="${-pi/2} 0 ${-pi/2}"/>
-      <parent link="camera_mount_link"/>
-      <child link="camera_optical_link"/>
+      <parent link="${robot_name}/camera_mount_link"/>
+      <child link="${robot_name}/camera_optical_link"/>
   </joint>
 </robot>

File: slambot_description/urdf/modules/chassis_and_wheels.xacro (robot description, xacro)
@@ -5,13 +5,13 @@
 <!-- THIS WAS ADDED IN MANUALLY -->
 <!-- Link base footprint -->
-<link name="base_footprint"/>
+<link name="${robot_name}/base_footprint"/>
 <!-- Joint base footprint -->
-<joint name="base_joint" type="fixed">
-    <parent link="base_footprint" />
-    <child link="chassis_link" />
+<joint name="${robot_name}/base_joint" type="fixed">
+    <parent link="${robot_name}/base_footprint" />
+    <child link="${robot_name}/chassis_link" />
     <origin xyz="0 0 0.045" rpy="0 0 0" />
 </joint>
 <!-- Link chassis -->
-  <link name="chassis_link">
+  <link name="${robot_name}/chassis_link">
     <inertial>
       <origin xyz="-0.00515019 1.96522e-17 0.0424366" rpy="0 0 0"/>
@@ -37,5 +37,5 @@
   </link>
   <!-- Link caster_frame -->
-  <link name="caster_frame_link">
+  <link name="${robot_name}/caster_frame_link">
     <inertial>
       <origin xyz="-0.0029329 -8.67362e-19 0.0118246" rpy="0 0 0"/>
@@ -61,5 +61,5 @@
   </link>
   <!-- Link caster_wheel -->
-  <link name="caster_wheel_link">
+  <link name="${robot_name}/caster_wheel_link">
     <inertial>
       <origin xyz="0 -1.22647e-18 0.0085" rpy="0 0 0"/>
@@ -85,21 +85,21 @@
   </link>
   <!-- Joint from caster_frame to caster_wheel -->
-  <joint name="caster_wheel_joint" type="continuous">
+  <joint name="${robot_name}/caster_wheel_joint" type="continuous">
     <origin xyz="-0.0110526 0.0085 0.024" rpy="1.5708 -0 0"/>
-    <parent link="caster_frame_link"/>
-    <child link="caster_wheel_link"/>
+    <parent link="${robot_name}/caster_frame_link"/>
+    <child link="${robot_name}/caster_wheel_link"/>
     <axis xyz="0 0 1"/>
     <limit effort="100" velocity="100"/>
   </joint>
   <!-- Joint from chassis to caster_frame -->
-  <joint name="caster_frame_joint" type="continuous">
+  <joint name="${robot_name}/caster_frame_joint" type="continuous">
     <origin xyz="0.07 -1.04083e-17 -0.006" rpy="3.14159 -0 0"/>
-    <parent link="chassis_link"/>
-    <child link="caster_frame_link"/>
+    <parent link="${robot_name}/chassis_link"/>
+    <child link="${robot_name}/caster_frame_link"/>
     <axis xyz="0 0 1"/>
     <limit effort="100" velocity="100"/>
   </joint>
   <!-- Link right_wheel -->
-  <link name="right_wheel_link">
+  <link name="${robot_name}/right_wheel_link">
     <inertial>
       <origin xyz="-2.40006e-17 1.14016e-17 0.0247872" rpy="0 0 0"/>
@@ -125,13 +125,13 @@
   </link>
   <!-- Joint from chassis to right_wheel -->
-  <joint name="right_wheel_joint" type="continuous">
+  <joint name="${robot_name}/right_wheel_joint" type="continuous">
     <origin xyz="-0.0561509 -0.0415 -0.01" rpy="1.5708 -0 0"/>
-    <parent link="chassis_link"/>
-    <child link="right_wheel_link"/>
+    <parent link="${robot_name}/chassis_link"/>
+    <child link="${robot_name}/right_wheel_link"/>
     <axis xyz="0 0 -1"/>
     <limit effort="100" velocity="100"/>
   </joint>
   <!-- Link left_wheel -->
-  <link name="left_wheel_link">
+  <link name="${robot_name}/left_wheel_link">
     <inertial>
       <origin xyz="-2.40006e-17 1.14016e-17 0.0247872" rpy="0 0 0"/>
@@ -157,8 +157,8 @@
   </link>
   <!-- Joint from chassis to left_wheel -->
-  <joint name="left_wheel_joint" type="continuous">
+  <joint name="${robot_name}/left_wheel_joint" type="continuous">
     <origin xyz="-0.0561509 0.0415 -0.01" rpy="-1.5708 -0 0"/>
-    <parent link="chassis_link"/>
-    <child link="left_wheel_link"/>
+    <parent link="${robot_name}/chassis_link"/>
+    <child link="${robot_name}/left_wheel_link"/>
     <axis xyz="0 0 1"/>
     <limit effort="100" velocity="100"/>

File: slambot_description/urdf/modules/lidar.xacro (robot description, xacro)
@@ -4,5 +4,5 @@
 <robot xmlns:xacro="http://www.ros.org/wiki/xacro">
  <!-- Link lidar -->
-  <link name="lidar_link">
+  <link name="${robot_name}/lidar_link">
     <inertial>
       <origin xyz="1.0786e-18 -3.85186e-34 -0.0125" rpy="0 0 0"/>
@@ -28,8 +28,8 @@
   </link>
   <!-- Joint from chassis to lidar -->
-  <joint name="lidar_joint" type="fixed">
+  <joint name="${robot_name}/lidar_joint" type="fixed">
     <origin xyz="-2.08167e-17 -8.72618e-18 0.072" rpy="3.14159 -0 0"/>
-    <parent link="chassis_link"/>
-    <child link="lidar_link"/>
+    <parent link="${robot_name}/chassis_link"/>
+    <child link="${robot_name}/lidar_link"/>
     <axis xyz="0 0 1"/>
     <limit effort="100" velocity="100"/>
