Commit message: update to the urdf to match the physical slambot dimensions, weights etc.

File: slambot_description/urdf/gazebo/gazebo_plugins.xacro (robot description, xacro)
@@ -11,6 +11,6 @@
             <right_joint>rear_right_wheel_joint</right_joint>
             <!--kinematics-->
-            <wheel_separation>0.147</wheel_separation>
-            <wheel_radius>0.03</wheel_radius>
+            <wheel_separation>0.198</wheel_separation>
+            <wheel_radius>0.034</wheel_radius>
             <!--limits-->
             <max_linear_acceleration>10</max_linear_acceleration>

File: slambot_description/urdf/modules/camera.xacro (robot description, xacro)
@@ -4,20 +4,20 @@
   <link name="camera_link">
     <inertial>
-      <origin xyz="1.31869e-19 -1.51987e-19 -0.00371932" rpy="0 0 0"/>
-      <mass value="0.000522865"/>
-      <inertia ixx="4.84738e-09" ixy="0" ixz="0" iyy="4.84738e-09" iyz="0" izz="4.86692e-09"/>
+      <origin xyz="5.37582e-18 -7.20266e-19 -0.0175" rpy="0 0 0"/>
+      <mass value="0.0229688"/>
+      <inertia ixx="4.68945e-06" ixy="0" ixz="0" iyy="2.77539e-06" iyz="0" izz="2.77539e-06"/>
     </inertial>
     <!-- Part camera_link -->
     <visual>
-      <origin xyz="0 3.85494e-19 0" rpy="3.14159 -0 0"/>
+      <origin xyz="6.45358e-18 0 -0.0175" rpy="3.14159 -0 0"/>
       <geometry>
         <mesh filename="package://slambot_description/assets/camera_link.stl"/>
       </geometry>
       <material name="camera_link_material">
-        <color rgba="0.980392 0.713725 0.00392157 1"/>
+        <color rgba="0.972549 0.529412 0.00392157 1"/>
       </material>
     </visual>
     <collision>
-      <origin xyz="0 3.85494e-19 0" rpy="3.14159 -0 0"/>
+      <origin xyz="6.45358e-18 0 -0.0175" rpy="3.14159 -0 0"/>
       <geometry>
         <mesh filename="package://slambot_description/assets/camera_link.stl"/>
@@ -26,6 +26,6 @@
   </link>
   <!-- Joint from base_link to camera_link -->
-  <joint name="camera_joint" type="fixed">
-    <origin xyz="0.0811976 3.85494e-19 0.057" rpy="0 -0 0"/>
+  <joint name="camera" type="fixed">
+    <origin xyz="0.083 -2.43306e-17 0.095" rpy="0 -0 0"/>
     <parent link="base_link"/>
     <child link="camera_link"/>
@@ -33,5 +33,5 @@
     <limit effort="100" velocity="100"/>
   </joint>
-    <!--THIS IS A FIX TO CHANGE THE ORIENTATION SO IT WORKS WITH OPENCV (ALWAYS INCLUDE)
+<!--THIS IS A FIX TO CHANGE THE ORIENTATION SO IT WORKS WITH OPENCV (ALWAYS INCLUDE)
   generate an optical frame
   http://www.ros.org/reps/rep-0103.html#suffix-frames

File: slambot_description/urdf/modules/chassis_and_wheels.xacro (robot description, xacro)
@@ -7,12 +7,12 @@
       <parent link="base_footprint" />
       <child link="base_link" />
-      <origin xyz="0 0 0.004" rpy="0 0 0" />
+      <origin xyz="0 0 0.019" rpy="0 0 0" />
   </joint>
-  <!-- Link base_link -->
+<!-- Link base_link -->
   <link name="base_link">
     <inertial>
-      <origin xyz="-0.00978934 8.10483e-16 0.0392801" rpy="0 0 0"/>
-      <mass value="2.10059"/>
-      <inertia ixx="0.00360353" ixy="0" ixz="0.000635006" iyy="0.00682291" iyz="0" izz="0.00795693"/>
+      <origin xyz="-0.00178426 -0.000464244 0.021065" rpy="0 0 0"/>
+      <mass value="1.56734"/>
+      <inertia ixx="0.0042106" ixy="1.29827e-06" ixz="0.000258451" iyy="0.0071422" iyz="5.95559e-06" izz="0.00967847"/>
     </inertial>
     <!-- Part base_link -->
@@ -23,5 +23,5 @@
       </geometry>
       <material name="base_link_material">
-        <color rgba="0.231373 0.380392 0.705882 1"/>
+        <color rgba="1 0 0 1"/>
       </material>
     </visual>
@@ -36,20 +36,20 @@
   <link name="rear_right_wheel_link">
     <inertial>
-      <origin xyz="-8.65114e-09 5.12286e-09 -0.0132554" rpy="0 0 0"/>
-      <mass value="0.0478503"/>
-      <inertia ixx="1.60159e-05" ixy="-2.44085e-12" ixz="-8.19615e-12" iyy="1.60159e-05" iyz="1.09538e-11" izz="2.75064e-05"/>
+      <origin xyz="-9.27276e-19 2.38145e-18 0.0198476" rpy="0 0 0"/>
+      <mass value="0.0642702"/>
+      <inertia ixx="2.85888e-05" ixy="-1.90555e-11" ixz="0" iyy="2.85888e-05" iyz="0" izz="4.92789e-05"/>
     </inertial>
     <!-- Part rear_right_wheel_link -->
     <visual>
-      <origin xyz="0 0 -0.0235" rpy="1.5708 -0 0"/>
+      <origin xyz="0 0 0.032" rpy="-1.5708 -0 0"/>
       <geometry>
         <mesh filename="package://slambot_description/assets/wheel_link.stl"/>
       </geometry>
       <material name="wheel_link_material">
-        <color rgba="0.647059 0.647059 0.647059 1"/>
+        <color rgba="0.901961 0.901961 0.901961 1"/>
       </material>
     </visual>
     <collision>
-      <origin xyz="0 0 -0.0235" rpy="1.5708 -0 0"/>
+      <origin xyz="0 0 0.032" rpy="-1.5708 -0 0"/>
       <geometry>
         <mesh filename="package://slambot_description/assets/wheel_link.stl"/>
@@ -59,8 +59,8 @@
   <!-- Joint from base_link to rear_right_wheel_link -->
   <joint name="rear_right_wheel_joint" type="continuous">
-    <origin xyz="-0.075 -0.06 0.02" rpy="-1.5708 -0 0"/>
+    <origin xyz="-0.0825 -0.08 0.015" rpy="1.5708 -0 0"/>
     <parent link="base_link"/>
     <child link="rear_right_wheel_link"/>
-    <axis xyz="0 0 1"/>
+    <axis xyz="0 0 -1"/>
     <limit effort="100" velocity="100"/>
   </joint>
@@ -68,20 +68,20 @@
   <link name="front_right_wheel_link">
     <inertial>
-      <origin xyz="-8.65114e-09 5.12286e-09 -0.0132554" rpy="0 0 0"/>
-      <mass value="0.0478503"/>
-      <inertia ixx="1.60159e-05" ixy="-2.44085e-12" ixz="-8.19615e-12" iyy="1.60159e-05" iyz="1.09538e-11" izz="2.75064e-05"/>
+      <origin xyz="-9.27276e-19 -2.38145e-18 -0.0198476" rpy="0 0 0"/>
+      <mass value="0.0642702"/>
+      <inertia ixx="2.85888e-05" ixy="1.90555e-11" ixz="0" iyy="2.85888e-05" iyz="0" izz="4.92789e-05"/>
     </inertial>
     <!-- Part front_right_wheel_link -->
     <visual>
-      <origin xyz="0 0 -0.0235" rpy="1.5708 -0 0"/>
+      <origin xyz="0 0 -0.032" rpy="1.5708 -0 0"/>
       <geometry>
         <mesh filename="package://slambot_description/assets/wheel_link.stl"/>
       </geometry>
       <material name="wheel_link_2_material">
-        <color rgba="0.647059 0.647059 0.647059 1"/>
+        <color rgba="0.901961 0.901961 0.901961 1"/>
       </material>
     </visual>
     <collision>
-      <origin xyz="0 0 -0.0235" rpy="1.5708 -0 0"/>
+      <origin xyz="0 0 -0.032" rpy="1.5708 -0 0"/>
       <geometry>
         <mesh filename="package://slambot_description/assets/wheel_link.stl"/>
@@ -91,5 +91,5 @@
   <!-- Joint from base_link to front_right_wheel_link -->
   <joint name="front_right_wheel_joint" type="continuous">
-    <origin xyz="0.075 -0.06 0.02" rpy="-1.5708 -0 0"/>
+    <origin xyz="0.0825 -0.08 0.015" rpy="-1.5708 -0 0"/>
     <parent link="base_link"/>
     <child link="front_right_wheel_link"/>
@@ -97,23 +97,55 @@
     <limit effort="100" velocity="100"/>
   </joint>
-  <!-- Link rear_left_wheel_link -->
-  <link name="rear_left_wheel_link">
+  <!-- Link front_left_wheel_link -->
+  <link name="front_left_wheel_link">
     <inertial>
-      <origin xyz="-8.65114e-09 -5.12286e-09 0.0132554" rpy="0 0 0"/>
-      <mass value="0.0478503"/>
-      <inertia ixx="1.60159e-05" ixy="2.44085e-12" ixz="8.19615e-12" iyy="1.60159e-05" iyz="1.09538e-11" izz="2.75064e-05"/>
+      <origin xyz="-9.27276e-19 -2.38145e-18 -0.0198476" rpy="0 0 0"/>
+      <mass value="0.0642702"/>
+      <inertia ixx="2.85888e-05" ixy="1.90555e-11" ixz="0" iyy="2.85888e-05" iyz="0" izz="4.92789e-05"/>
     </inertial>
-    <!-- Part rear_left_wheel_link -->
+    <!-- Part front_left_wheel_link -->
     <visual>
-      <origin xyz="0 0 0.0235" rpy="-1.5708 -0 0"/>
+      <origin xyz="0 0 -0.032" rpy="1.5708 -0 0"/>
       <geometry>
         <mesh filename="package://slambot_description/assets/wheel_link.stl"/>
       </geometry>
       <material name="wheel_link_3_material">
-        <color rgba="0.647059 0.647059 0.647059 1"/>
+        <color rgba="0.901961 0.901961 0.901961 1"/>
       </material>
     </visual>
     <collision>
-      <origin xyz="0 0 0.0235" rpy="-1.5708 -0 0"/>
+      <origin xyz="0 0 -0.032" rpy="1.5708 -0 0"/>
+      <geometry>
+        <mesh filename="package://slambot_description/assets/wheel_link.stl"/>
+      </geometry>
+    </collision>
+  </link>
+  <!-- Joint from base_link to front_left_wheel_link -->
+  <joint name="front_left_wheel_joint" type="continuous">
+    <origin xyz="0.0825 0.08 0.015" rpy="1.5708 -0 0"/>
+    <parent link="base_link"/>
+    <child link="front_left_wheel_link"/>
+    <axis xyz="0 0 -1"/>
+    <limit effort="100" velocity="100"/>
+  </joint>
+  <!-- Link rear_left_wheel_link -->
+  <link name="rear_left_wheel_link">
+    <inertial>
+      <origin xyz="-9.27276e-19 2.38145e-18 0.0198476" rpy="0 0 0"/>
+      <mass value="0.0642702"/>
+      <inertia ixx="2.85888e-05" ixy="-1.90555e-11" ixz="0" iyy="2.85888e-05" iyz="0" izz="4.92789e-05"/>
+    </inertial>
+    <!-- Part rear_left_wheel_link -->
+    <visual>
+      <origin xyz="0 0 0.032" rpy="-1.5708 -0 0"/>
+      <geometry>
+        <mesh filename="package://slambot_description/assets/wheel_link.stl"/>
+      </geometry>
+      <material name="wheel_link_4_material">
+        <color rgba="0.901961 0.901961 0.901961 1"/>
+      </material>
+    </visual>
+    <collision>
+      <origin xyz="0 0 0.032" rpy="-1.5708 -0 0"/>
       <geometry>
         <mesh filename="package://slambot_description/assets/wheel_link.stl"/>
@@ -123,5 +155,5 @@
   <!-- Joint from base_link to rear_left_wheel_link -->
   <joint name="rear_left_wheel_joint" type="continuous">
-    <origin xyz="-0.075 0.06 0.02" rpy="-1.5708 -0 0"/>
+    <origin xyz="-0.0825 0.08 0.015" rpy="-1.5708 -0 0"/>
     <parent link="base_link"/>
     <child link="rear_left_wheel_link"/>
@@ -129,35 +161,3 @@
     <limit effort="100" velocity="100"/>
   </joint>
-  <!-- Link front_left_wheel_link -->
-  <link name="front_left_wheel_link">
-    <inertial>
-      <origin xyz="-8.65114e-09 -5.12286e-09 0.0132554" rpy="0 0 0"/>
-      <mass value="0.0478503"/>
-      <inertia ixx="1.60159e-05" ixy="2.44085e-12" ixz="8.19615e-12" iyy="1.60159e-05" iyz="1.09538e-11" izz="2.75064e-05"/>
-    </inertial>
-    <!-- Part front_left_wheel_link -->
-    <visual>
-      <origin xyz="0 0 0.0235" rpy="-1.5708 -0 0"/>
-      <geometry>
-        <mesh filename="package://slambot_description/assets/wheel_link.stl"/>
-      </geometry>
-      <material name="wheel_link_4_material">
-        <color rgba="0.647059 0.647059 0.647059 1"/>
-      </material>
-    </visual>
-    <collision>
-      <origin xyz="0 0 0.0235" rpy="-1.5708 -0 0"/>
-      <geometry>
-        <mesh filename="package://slambot_description/assets/wheel_link.stl"/>
-      </geometry>
-    </collision>
-  </link>
-  <!-- Joint from base_link to front_left_wheel_link -->
-  <joint name="front_left_wheel_joint" type="continuous">
-    <origin xyz="0.075 0.06 0.02" rpy="-1.5708 -0 0"/>
-    <parent link="base_link"/>
-    <child link="front_left_wheel_link"/>
-    <axis xyz="0 0 1"/>
-    <limit effort="100" velocity="100"/>
-  </joint>
 </robot>

File: slambot_description/urdf/modules/imu.xacro (robot description, xacro)
@@ -8,5 +8,5 @@
     <child link="imu_link"/>
     <!-- Place the IMU physically on the base_link, you can adjust the xyz values -->
-    <origin xyz="0 0 0.05" rpy="0 0 0"/>
+    <origin xyz="0 0 0.06" rpy="0 0 0"/>
   </joint>
 </robot>

File: slambot_description/urdf/modules/lidar.xacro (robot description, xacro)
@@ -4,20 +4,20 @@
   <link name="lidar_link">
     <inertial>
-      <origin xyz="-1.11789e-18 1.22638e-20 -0.00745144" rpy="0 0 0"/>
-      <mass value="0.0267087"/>
-      <inertia ixx="4.66132e-06" ixy="0" ixz="0" iyy="4.66132e-06" iyz="0" izz="8.33295e-06"/>
+      <origin xyz="-1.06386e-18 5.77779e-34 -0.0125" rpy="0 0 0"/>
+      <mass value="0.041469"/>
+      <inertia ixx="6.30675e-06" ixy="0" ixz="0" iyy="6.30675e-06" iyz="0" izz="8.2938e-06"/>
     </inertial>
     <!-- Part lidar_link -->
     <visual>
-      <origin xyz="0 1.53081e-18 0" rpy="3.14159 -0 0"/>
+      <origin xyz="0 1.22465e-18 0" rpy="3.14159 -0 0"/>
       <geometry>
         <mesh filename="package://slambot_description/assets/lidar_link.stl"/>
       </geometry>
       <material name="lidar_link_material">
-        <color rgba="0.301961 0.301961 0.301961 1"/>
+        <color rgba="0 0 0 1"/>
       </material>
     </visual>
     <collision>
-      <origin xyz="0 1.53081e-18 0" rpy="3.14159 -0 0"/>
+      <origin xyz="0 1.22465e-18 0" rpy="3.14159 -0 0"/>
       <geometry>
         <mesh filename="package://slambot_description/assets/lidar_link.stl"/>
@@ -26,7 +26,7 @@
   </link>
   <!-- Joint from base_link to lidar_link -->
-  <joint name="lidar_joint" type="fixed">
-    <!--<origin xyz="-0.0440219 2.92864e-17 0.09" rpy="3.14159 -0 0"/>--> <!--Changed because lidar z-axis was actually pointing DOWN!-->
-    <origin xyz="-0.0440219 2.92864e-17 0.105" rpy="0 -0 0"/>
+  <joint name="lidar" type="fixed">
+    <!--<origin xyz="-0.050039 8.16354e-18 0.105" rpy="3.14159 -0 0"/>-->
+    <origin xyz="-0.050039 8.16354e-18 0.13" rpy="0 -0 0"/>  <!-- If z-axis pointing down, use this instead-->
     <parent link="base_link"/>
     <child link="lidar_link"/>
